File: snickerdoodle.kicad_sch (KiCad schematic)
At the start: 7 parts, among them P2 TFM-115-01-F-D-A, P3 TFM-120-01-F-D-A

Commit message: Fix bus names, add I2C, add footprints and 3D models
Parts:
- P2: footprint (none) -> Connector_Samtec_TFM:Samtec_TFM-115-01-F-D-A_2x15_P1.27mm_Horizontal
- P3, PA1, PA2, PB1, PB2, PC1: footprint (none) -> Connector_Samtec_TFM:Samtec_TFM-120-01-F-D-A_2x20_P1.27mm_Horizontal
Connections:
- net JC.~INT1: now reaches PC1.2 (Pin_2)
- net ZYNQ_I2C4.SCL: now reaches PC1.39 (Pin_39)
- net ZYNQ_I2C4.SDA: now reaches PC1.40 (Pin_40)
- net JB.~INT1: now reaches PB1.2 (Pin_2)
- net ZYNQ_I2C2.SCL: now reaches PB1.39 (Pin_39)
- net ZYNQ_I2C2.SDA: now reaches PB1.40 (Pin_40)
- net JA.~INT1: now reaches PA1.2 (Pin_2)
- net ZYNQ_I2C0.SCL: now reaches PA1.39 (Pin_39)
- net ZYNQ_I2C0.SDA: now reaches PA1.40 (Pin_40)
- net JA.~INT2: now reaches PA2.2 (Pin_2)
- net ZYNQ_I2C1.SCL: now reaches PA2.39 (Pin_39)
- net ZYNQ_I2C1.SDA: now reaches PA2.40 (Pin_40)
- net 3.3V_VIO: now reaches P2.25 (Pin_25)
- net ZYNQ_I2C7.SCL: now reaches P2.7 (Pin_7)
- net ZYNQ_I2C7.SDA: now reaches P2.8 (Pin_8)
- net ZYNQ_I2C5.SCL: now reaches P3.39 (Pin_39)
- net ZYNQ_I2C5.SDA: now reaches P3.40 (Pin_40)
- net JB.~INT2: now reaches PB2.2 (Pin_2)
- net ZYNQ_I2C3.SCL: now reaches PB2.39 (Pin_39)
- net ZYNQ_I2C3.SDA: now reaches PB2.40 (Pin_40)
- net FPGA_VIN renamed ZYNQ_VIN
- net JTAG.PGND renamed PGND
- net JTAG.TCK renamed TCK
- net JTAG.TDI renamed TDI
- net JTAG.TDO renamed TDO
- net JTAG.TMS renamed TMS
- net JTAG.~RST renamed ZYNQ_~RST
- net SWD.CLK renamed SWCLK
- net SWD.IO renamed SWDIO
- net SWD.~RST renamed MCU_~RST
Other:
- note added: "ZYNQ_VIN should be between +3.7 and +17V."
- note removed: "FPGA_VIN should be between +3.7 and +17V."

Commit message: Layout connectors on PCB
Parts:
- added H1: MountingHole, Snickerdoodle:Snickerdoodle_Mounting_Hole, symbol Mechanical:MountingHole
Changed lines of the file:
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@@
 (kicad_sch (version 20200608) (host eeschema "5.99.0-unknown-ad69e44~101~ubuntu20.04.1")
-  (page 3 2)
+  (page 2 2)
   (paper "A4")
   (title_block
@@
   (symbol (lib_id "Snickerdoodle:3.3V_VIO") (at 182.88 134.62 0)
     (in_bom yes) (on_board yes)
-    (property "Reference" "#PWR?" (id 0) (at 182.88 138.43 0)
+    (property "Reference" "#PWR0115" (id 0) (at 182.88 138.43 0)
       (effects (font (size 1.27 1.27)) hide)
     )
@@
       (effects (font (size 1.27 1.27)) hide)
     )
+  )
+  (symbol (lib_id "Mechanical:MountingHole") (at 254 152.4 0) (unit 1)
+    (in_bom yes) (on_board yes)
+    (property "Reference" "H1" (id 0) (at 256.5401 151.2506 0)
+      (effects (font (size 1.27 1.27)) (justify left))
+    )
+    (property "Value" "MountingHole" (id 1) (at 256.5401 153.5493 0)
+      (effects (font (size 1.27 1.27)) (justify left))
+    )
+    (property "Footprint" "Snickerdoodle:Snickerdoodle_Mounting_Hole" (id 2) (at 254 152.4 0)
+      (effects (font (size 1.27 1.27)) hide)
+    )
+    (property "Datasheet" "~" (id 3) (at 254 152.4 0)
+      (effects (font (size 1.27 1.27)) hide)
+    )
